Commit message: axis positioning issue

File: urdf/diff_drive.xacro (robot description, xacro)
@@ -97,5 +97,5 @@
         <parent link="base_link" />
         <child link="right_wheel_1" />
-        <axis xyz="0.0 -1.0 0.0" />
+        <axis xyz="0.0 1.0 0.0" />
     </joint>
     <joint name="Revolute_2" type="continuous">
